Commit message: Add files via upload

File: src/simu_bipo/description/arobot.urdf.xacro (robot description, xacro)
@@ -3,4 +3,5 @@
     <xacro:include filename="bipo.xacro" />
     <xacro:include filename="gazebo_references.xacro" />
-    <xacro:include filename="ros2_control.xacro" />
+    <!-- SET THE CONTROLLER TO BE USED -->
+    <xacro:include filename="foward_position_controller.xacro" />
 </robot>

File: src/simu_bipo/description/bipo.xacro (robot description, xacro)
@@ -110,6 +110,6 @@
       velocity="100" />
     <dynamics
-      damping="0.1"
-      friction="0.1" />
+      damping="0.000001"
+      friction="0.000001" />
   </joint>
   <link
@@ -120,5 +120,5 @@
         rpy="0 0 0" />
       <mass
-        value="6.2077" />
+        value="1.0" />
       <inertia
         ixx="0.014538"
@@ -171,6 +171,6 @@
       velocity="100" />
     <dynamics
-      damping="0.1"
-      friction="0.1" />
+      damping="0.000001"
+      friction="0.000001" />
   </joint>
   <link
@@ -181,5 +181,5 @@
         rpy="0 0 0" />
       <mass
-        value="4.7184" />
+        value="3.861" />
       <inertia
         ixx="0.0083251"
@@ -232,6 +232,6 @@
       velocity="100" />
     <dynamics
-      damping="0.1"
-      friction="0.1" />
+      damping="0.000001"
+      friction="0.000001" />
   </joint>
   <link
@@ -242,5 +242,5 @@
         rpy="0 0 0" />
       <mass
-        value="1.1717" />
+        value="0.78" />
       <inertia
         ixx="0.00046552"
@@ -293,6 +293,6 @@
       velocity="100" />
     <dynamics
-      damping="0.1"
-      friction="0.1" />
+      damping="0.000001"
+      friction="0.000001" />
   </joint>
   <link
@@ -303,5 +303,5 @@
         rpy="0 0 0" />
       <mass
-        value="0.23479" />
+        value="0.254" />
       <inertia
         ixx="0.0000504"
@@ -354,5 +354,5 @@
       velocity="100" />
     <dynamics
-      damping="0.1"
+      damping="0.000001"
       friction="0.1" />
   </joint>
@@ -364,5 +364,5 @@
         rpy="0 0 0" />
       <mass
-        value="1.1717" />
+        value="0.78" />
       <inertia
         ixx="0.00046552"
@@ -415,6 +415,6 @@
       velocity="100" />
     <dynamics
-      damping="0.1"
-      friction="0.1" />
+      damping="0.000001"
+      friction="0.000001" />
   </joint>
   <link
@@ -425,5 +425,5 @@
         rpy="0 0 0" />
       <mass
-        value="0.23479" />
+        value="0.254" />
       <inertia
         ixx="0.0000504"
@@ -476,6 +476,6 @@
       velocity="100" />
     <dynamics
-      damping="0.1"
-      friction="0.1" />
+      damping="0.000001"
+      friction="10" />
   </joint>
 </robot>

File: src/simu_bipo/description/gazebo_references.xacro (robot description, xacro)
@@ -3,40 +3,40 @@
   <gazebo reference="L_0_link">
     <material>Gazebo/Gray</material>
-    <mu1>0.001</mu1>
+    <mu1>0.01</mu1>
     <mu2>0.001</mu2>
   </gazebo>
   <gazebo reference="L_1_link">
-    <material>Gazebo/Gray</material>
-    <mu1>0.001</mu1>
+    <material>Gazebo/Green</material>
+    <mu1>0.01</mu1>
     <mu2>0.001</mu2>
   </gazebo>
   <gazebo reference="L_2_link">
     <material>Gazebo/Gray</material>
-    <mu1>0.001</mu1>
+    <mu1>0.01</mu1>
     <mu2>0.001</mu2>
   </gazebo>
   <gazebo reference="L_3_link">
     <material>Gazebo/Gray</material>
-    <mu1>0.001</mu1>
+    <mu1>0.01</mu1>
     <mu2>0.001</mu2>
   </gazebo>
   <gazebo reference="L_4_link">
     <material>Gazebo/Gray</material>
-    <mu1>0.001</mu1>
+    <mu1>0.01</mu1>
     <mu2>0.001</mu2>
   </gazebo>
   <gazebo reference="L_5_link">
-    <material>Gazebo/Gray</material>
-    <mu1>0.001</mu1>
+    <material>Gazebo/Green</material>
+    <mu1>0.01</mu1>
     <mu2>0.001</mu2>
   </gazebo>
   <gazebo reference="L_6_link">
     <material>Gazebo/Gray</material>
-    <mu1>0.001</mu1>
+    <mu1>0.01</mu1>
     <mu2>0.001</mu2>
   </gazebo>
   <gazebo reference="L_7_link">
     <material>Gazebo/Gray</material>
-    <mu1>0.001</mu1>
+    <mu1>0.01</mu1>
     <mu2>0.001</mu2>
   </gazebo>
